File: hw/n64cart.brd (EAGLE design)
At the start: 99.1 x 50.8 mm, 38 parts, among them IC1 RP2040-QFN56, J1 N64_EDGE, Q1 BSS84, U1 W25Q128JVSIQ, U3 W25Q256JVEIQ_TR

Commit message: added capacitor to VBUS
Parts:
- added C4: 100n, rcl:C0402
Connections:
- net +VBUS: now also C4.1
- net GND: now also C4.2
Routing:
- net +VBUS: track 22.0 -> 24.4 mm
Changed lines of the file:
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@@
 <attribute name="VALUE" x="50.47503125" y="33.71476875" size="1.27135" layer="27" rot="R180"/>
+</element>
+<element name="C4" library="rcl" library_urn="urn:adsk.eagle:library:334" package="C0402" package3d_urn="urn:adsk.eagle:package:23626/2" value="100n" x="11.43" y="50.8" smashed="yes" rot="R180">
+<attribute name="NAME" x="12.065" y="52.705" size="1.27" layer="25" rot="R180"/>
+<attribute name="POPULARITY" value="18" x="11.43" y="50.8" size="1.778" layer="27" rot="R180" display="off"/>
+<attribute name="SPICEPREFIX" value="C" x="11.43" y="50.8" size="1.778" layer="27" rot="R180" display="off"/>
+<attribute name="VALUE" x="12.065" y="52.705" size="1.27" layer="27" rot="R180"/>
 </element>
 </elements>
@@
 <via x="68.58" y="45.72" extent="1-16" drill="0.35"/>
 <via x="50.038" y="35.687" extent="1-16" drill="0.35"/>
+<contactref element="C4" pad="2"/>
 </signal>
 <signal name="+3V3">
@@
 <contactref element="Q1" pad="1"/>
 <contactref element="U$1" pad="3"/>
-<wire x1="3.97" y1="49.56" x2="14.6" y2="49.56" width="0.3048" layer="1"/>
+<wire x1="3.97" y1="49.56" x2="13.97" y2="49.56" width="0.3048" layer="1"/>
+<wire x1="13.97" y1="49.56" x2="14.6" y2="49.56" width="0.3048" layer="1"/>
 <wire x1="14.6" y1="49.56" x2="14.86" y2="49.3" width="0.3048" layer="1"/>
 <wire x1="14.86" y1="49.3" x2="25.32" y2="49.3" width="0.3048" layer="1"/>
 <wire x1="25.32" y1="49.3" x2="25.72" y2="49.7" width="0.3048" layer="1"/>
+<contactref element="C4" pad="1"/>
+<wire x1="12.08" y1="50.8" x2="12.73" y2="50.8" width="0.3048" layer="1"/>
+<wire x1="12.73" y1="50.8" x2="13.97" y2="49.56" width="0.3048" layer="1"/>
 </signal>
 <signal name="SWCLK">

Commit message: latest version
Parts:
- added C7: 100n, rcl:C0402
Connections:
- net GND: now also C7.2
- net N$1: now also C7.1
Routing:
- net N$1: track 3.83 -> 6.62 mm
Changed lines of the file:
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@@
 <attribute name="VALUE" x="12.065" y="52.705" size="1.27" layer="27" rot="R180"/>
+</element>
+<element name="C7" library="rcl" library_urn="urn:adsk.eagle:library:334" package="C0402" package3d_urn="urn:adsk.eagle:package:23626/2" value="100n" x="21.59" y="53.34" smashed="yes">
+<attribute name="NAME" x="20.955" y="53.975" size="1.27" layer="25"/>
+<attribute name="POPULARITY" value="18" x="21.59" y="53.34" size="1.778" layer="27" display="off"/>
+<attribute name="SPICEPREFIX" value="C" x="21.59" y="53.34" size="1.778" layer="27" display="off"/>
+<attribute name="VALUE" x="20.955" y="51.435" size="1.27" layer="27"/>
 </element>
 </elements>
@@
 <via x="50.038" y="35.687" extent="1-16" drill="0.35"/>
 <contactref element="C4" pad="2"/>
+<contactref element="C7" pad="2"/>
 </signal>
 <signal name="+3V3">
@@
 <contactref element="D1" pad="A"/>
 <wire x1="16.51" y1="50.8" x2="20.34" y2="50.8" width="0.3048" layer="1"/>
+<contactref element="C7" pad="1"/>
+<wire x1="20.94" y1="53.34" x2="20.34" y2="52.74" width="0.3048" layer="1"/>
+<wire x1="20.34" y1="52.74" x2="20.34" y2="50.8" width="0.3048" layer="1"/>
 </signal>
 <signal name="N$4">
