File: hw/n64cart.sch (EAGLE design)
At the start: 38 parts, among them IC1 RP2040-QFN56, J1 N64_EDGE, Q1 BSS84, U1 W25Q128JVSIQ, U3 W25Q256JVEIQ_TR

Commit message: added capacitor to VBUS
Parts:
- added C4: 100n, rcl:C-EUC0402
Connections:
- net +VBUS: now also C4.1
- net GND: now also C4.2
Changed lines of the file:
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@@
 <part name="GND26" library="supply1" library_urn="urn:adsk.eagle:library:371" deviceset="GND" device=""/>
 <part name="U3" library="W25Q256JVEIQ_TR" deviceset="W25Q256JVEIQ_TR" device=""/>
+<part name="C4" library="rcl" library_urn="urn:adsk.eagle:library:334" deviceset="C-EU" device="C0402" package3d_urn="urn:adsk.eagle:package:23626/2" value="100n"/>
+<part name="GND27" library="supply1" library_urn="urn:adsk.eagle:library:371" deviceset="GND" device=""/>
 </parts>
 <sheets>
@@
 <attribute name="NAME" x="375.9185" y="320.5495" size="2.540359375" layer="95"/>
 <attribute name="VALUE" x="375.9182" y="296.6696" size="2.540459375" layer="96"/>
+</instance>
+<instance part="C4" gate="G$1" x="469.9" y="388.62" smashed="yes">
+<attribute name="NAME" x="471.424" y="389.001" size="1.778" layer="95"/>
+<attribute name="VALUE" x="471.424" y="383.921" size="1.778" layer="96"/>
+</instance>
+<instance part="GND27" gate="1" x="469.9" y="378.46" smashed="yes">
+<attribute name="VALUE" x="467.36" y="375.92" size="1.778" layer="96"/>
 </instance>
 </instances>
@@
 <pinref part="R7" gate="G$1" pin="2"/>
 <wire x1="614.68" y1="302.26" x2="614.68" y2="307.34" width="0.1524" layer="91"/>
+</segment>
+<segment>
+<pinref part="GND27" gate="1" pin="GND"/>
+<pinref part="C4" gate="G$1" pin="2"/>
+<wire x1="469.9" y1="381" x2="469.9" y2="383.54" width="0.1524" layer="91"/>
 </segment>
 </net>
@@
 <segment>
 <pinref part="U$1" gate="A" pin="VIN"/>
-<wire x1="472.44" y1="396.24" x2="464.82" y2="396.24" width="0.1524" layer="91"/>
+<wire x1="472.44" y1="396.24" x2="469.9" y2="396.24" width="0.1524" layer="91"/>
 <label x="464.82" y="396.24" size="1.27" layer="95" rot="R180" xref="yes"/>
-</segment>
-</net>
+<pinref part="C4" gate="G$1" pin="1"/>
+<wire x1="469.9" y1="396.24" x2="464.82" y2="396.24" width="0.1524" layer="91"/>
+<wire x1="469.9" y1="391.16" x2="469.9" y2="396.24" width="0.1524" layer="91"/>
+<junction x="469.9" y="396.24"/>
+</segment>
+</net>

Commit message: latest version
Parts:
- added C7: 100n, rcl:C-EUC0402
Connections:
- net GND: now also C7.2
- net N$1: now also C7.1
Changed lines of the file:
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@@
 <part name="C4" library="rcl" library_urn="urn:adsk.eagle:library:334" deviceset="C-EU" device="C0402" package3d_urn="urn:adsk.eagle:package:23626/2" value="100n"/>
 <part name="GND27" library="supply1" library_urn="urn:adsk.eagle:library:371" deviceset="GND" device=""/>
+<part name="C7" library="rcl" library_urn="urn:adsk.eagle:library:334" deviceset="C-EU" device="C0402" package3d_urn="urn:adsk.eagle:package:23626/2" value="100n"/>
 </parts>
 <sheets>
@@
 <attribute name="VALUE" x="477.5186" y="386.0773" size="1.77848125" layer="96"/>
 </instance>
-<instance part="GND25" gate="1" x="505.46" y="383.54" smashed="yes">
-<attribute name="VALUE" x="502.92" y="381" size="1.778" layer="96"/>
+<instance part="GND25" gate="1" x="505.46" y="378.46" smashed="yes">
+<attribute name="VALUE" x="502.92" y="375.92" size="1.778" layer="96"/>
 </instance>
 <instance part="D1" gate="G$1" x="515.62" y="396.24" smashed="yes">
@@
 <instance part="GND27" gate="1" x="469.9" y="378.46" smashed="yes">
 <attribute name="VALUE" x="467.36" y="375.92" size="1.778" layer="96"/>
+</instance>
+<instance part="C7" gate="G$1" x="510.54" y="391.16" smashed="yes">
+<attribute name="NAME" x="512.064" y="391.541" size="1.778" layer="95"/>
+<attribute name="VALUE" x="512.064" y="386.461" size="1.778" layer="96"/>
 </instance>
 </instances>
@@
 <pinref part="GND25" gate="1" pin="GND"/>
 <wire x1="502.92" y1="391.16" x2="505.46" y2="391.16" width="0.1524" layer="91"/>
-<wire x1="505.46" y1="391.16" x2="505.46" y2="386.08" width="0.1524" layer="91"/>
+<wire x1="505.46" y1="391.16" x2="505.46" y2="383.54" width="0.1524" layer="91"/>
+<pinref part="C7" gate="G$1" pin="2"/>
+<wire x1="505.46" y1="383.54" x2="505.46" y2="381" width="0.1524" layer="91"/>
+<wire x1="510.54" y1="386.08" x2="510.54" y2="383.54" width="0.1524" layer="91"/>
+<wire x1="510.54" y1="383.54" x2="505.46" y2="383.54" width="0.1524" layer="91"/>
+<junction x="505.46" y="383.54"/>
 </segment>
 <segment>
@@
 <pinref part="U$1" gate="A" pin="VOUT"/>
 <pinref part="D1" gate="G$1" pin="A"/>
-<wire x1="502.92" y1="396.24" x2="513.08" y2="396.24" width="0.1524" layer="91"/>
-</segment>
-</net>
+<wire x1="502.92" y1="396.24" x2="510.54" y2="396.24" width="0.1524" layer="91"/>
+<pinref part="C7" gate="G$1" pin="1"/>
+<wire x1="510.54" y1="396.24" x2="513.08" y2="396.24" width="0.1524" layer="91"/>
+<wire x1="510.54" y1="393.7" x2="510.54" y2="396.24" width="0.1524" layer="91"/>
+<junction x="510.54" y="396.24"/>
+</segment>
+</net>

Commit message: schematic in pdf
Other:
- note added: "Do not solder Q1 if D2 is soldered. Use either D2 or Q1. Do not solder R1 and R6."
- moved on the sheet: C22, D2, Q1
Changed lines of the file:
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@@
 <wire x1="215.9" y1="248.92" x2="215.9" y2="365.76" width="0.1524" layer="97" style="longdash"/>
 <text x="215.9" y="368.3" size="3.81" layer="97">N64 Edge Connector</text>
+<text x="220.98" y="200.66" size="2.54" layer="91">Do not solder Q1 if D2 is soldered. Use either D2 or Q1.
+Do not solder R1 and R6.</text>
 </plain>
 <instances>
@@
 <attribute name="VALUE" x="218.44" y="251.46" size="1.778" layer="96"/>
 </instance>
-<instance part="Q1" gate="G$1" x="655.32" y="431.8" smashed="yes" rot="R90">
-<attribute name="NAME" x="655.32" y="434.34" size="1.778" layer="95" rot="R90"/>
-<attribute name="VALUE" x="657.86" y="434.34" size="1.778" layer="96" rot="R90"/>
+<instance part="Q1" gate="G$1" x="576.58" y="396.24" smashed="yes" rot="R90">
+<attribute name="NAME" x="576.58" y="398.78" size="1.778" layer="95" rot="R90"/>
+<attribute name="VALUE" x="579.12" y="398.78" size="1.778" layer="96" rot="R90"/>
 </instance>
 <instance part="LED1" gate="G$1" x="601.98" y="325.12" smashed="yes" rot="MR0">
@@
 <attribute name="VALUE" x="599.44" y="297.18" size="1.778" layer="96"/>
 </instance>
-<instance part="D2" gate="G$1" x="668.02" y="424.18" smashed="yes" rot="R180">
-<attribute name="NAME" x="665.48" y="426.72" size="1.778" layer="95"/>
-<attribute name="VALUE" x="668.02" y="421.64" size="1.778" layer="96" rot="R270"/>
-</instance>
-<instance part="C22" gate="G$1" x="660.4" y="416.56" smashed="yes">
-<attribute name="NAME" x="661.924" y="416.941" size="1.778" layer="95"/>
-<attribute name="VALUE" x="661.924" y="411.861" size="1.778" layer="96"/>
-</instance>
-<instance part="GND4" gate="1" x="660.4" y="403.86" smashed="yes">
-<attribute name="VALUE" x="657.86" y="401.32" size="1.778" layer="96"/>
+<instance part="D2" gate="G$1" x="589.28" y="388.62" smashed="yes" rot="R180">
+<attribute name="NAME" x="586.74" y="391.16" size="1.778" layer="95"/>
+<attribute name="VALUE" x="589.28" y="386.08" size="1.778" layer="96" rot="R270"/>
+</instance>
+<instance part="C22" gate="G$1" x="581.66" y="381" smashed="yes">
+<attribute name="NAME" x="583.184" y="381.381" size="1.778" layer="95"/>
+<attribute name="VALUE" x="583.184" y="376.301" size="1.778" layer="96"/>
+</instance>
+<instance part="GND4" gate="1" x="581.66" y="368.3" smashed="yes">
+<attribute name="VALUE" x="579.12" y="365.76" size="1.778" layer="96"/>
 </instance>
 <instance part="IC1" gate="IC$1" x="469.9" y="246.38" smashed="yes">
@@
 <pinref part="C22" gate="G$1" pin="2"/>
 <pinref part="GND4" gate="1" pin="GND"/>
-<wire x1="660.4" y1="411.48" x2="660.4" y2="406.4" width="0.1524" layer="91"/>
+<wire x1="581.66" y1="375.92" x2="581.66" y2="370.84" width="0.1524" layer="91"/>
 </segment>
 <segment>
@@
 <segment>
 <pinref part="D2" gate="G$1" pin="C"/>
-<wire x1="665.48" y1="424.18" x2="660.4" y2="424.18" width="0.1524" layer="91"/>
+<wire x1="586.74" y1="388.62" x2="581.66" y2="388.62" width="0.1524" layer="91"/>
 <pinref part="C22" gate="G$1" pin="1"/>
-<wire x1="660.4" y1="419.1" x2="660.4" y2="424.18" width="0.1524" layer="91"/>
+<wire x1="581.66" y1="383.54" x2="581.66" y2="388.62" width="0.1524" layer="91"/>
 <pinref part="Q1" gate="G$1" pin="S"/>
-<wire x1="645.16" y1="424.18" x2="645.16" y2="431.8" width="0.1524" layer="91"/>
-<wire x1="645.16" y1="431.8" x2="650.24" y2="431.8" width="0.1524" layer="91"/>
-<wire x1="660.4" y1="424.18" x2="645.16" y2="424.18" width="0.1524" layer="91"/>
-<junction x="660.4" y="424.18"/>
-<wire x1="645.16" y1="431.8" x2="632.46" y2="431.8" width="0.1524" layer="91"/>
-<junction x="645.16" y="431.8"/>
-<label x="632.46" y="431.8" size="1.27" layer="95" rot="R180" xref="yes"/>
+<wire x1="566.42" y1="388.62" x2="566.42" y2="396.24" width="0.1524" layer="91"/>
+<wire x1="566.42" y1="396.24" x2="571.5" y2="396.24" width="0.1524" layer="91"/>
+<wire x1="581.66" y1="388.62" x2="566.42" y2="388.62" width="0.1524" layer="91"/>
+<junction x="581.66" y="388.62"/>
+<wire x1="566.42" y1="396.24" x2="553.72" y2="396.24" width="0.1524" layer="91"/>
+<junction x="566.42" y="396.24"/>
+<label x="553.72" y="396.24" size="1.27" layer="95" rot="R180" xref="yes"/>
 </segment>
 <segment>
@@
 <segment>
 <pinref part="Q1" gate="G$1" pin="D"/>
-<wire x1="665.48" y1="431.8" x2="660.4" y2="431.8" width="0.1524" layer="91"/>
-<label x="665.48" y="431.8" size="1.27" layer="95" xref="yes"/>
+<wire x1="586.74" y1="396.24" x2="581.66" y2="396.24" width="0.1524" layer="91"/>
+<label x="586.74" y="396.24" size="1.27" layer="95" xref="yes"/>
 </segment>
 <segment>
 <pinref part="D2" gate="G$1" pin="A"/>
-<wire x1="670.56" y1="424.18" x2="675.64" y2="424.18" width="0.1524" layer="91"/>
-<label x="675.64" y="424.18" size="1.27" layer="95" xref="yes"/>
+<wire x1="591.82" y1="388.62" x2="596.9" y2="388.62" width="0.1524" layer="91"/>
+<label x="596.9" y="388.62" size="1.27" layer="95" xref="yes"/>
 </segment>
 </net>
@@
 <segment>
 <pinref part="Q1" gate="G$1" pin="G"/>
-<wire x1="632.46" y1="416.56" x2="652.78" y2="416.56" width="0.1524" layer="91"/>
-<wire x1="652.78" y1="416.56" x2="652.78" y2="426.72" width="0.1524" layer="91"/>
-<label x="632.46" y="416.56" size="1.27" layer="95" rot="R180" xref="yes"/>
+<wire x1="553.72" y1="381" x2="574.04" y2="381" width="0.1524" layer="91"/>
+<wire x1="574.04" y1="381" x2="574.04" y2="391.16" width="0.1524" layer="91"/>
+<label x="553.72" y="381" size="1.27" layer="95" rot="R180" xref="yes"/>
 </segment>
 <segment>
@@
 </drawing>
 <compatibility>
+<note version="6.3" minversion="6.2.2" severity="warning">
+Since Version 6.2.2 text objects can contain more than one line,
+which will not be processed correctly with this version.
+</note>
 <note version="8.2" severity="warning">
 Since Version 8.2, EAGLE supports online libraries. The ids
