File: hw/n64cart-1G.sch (EAGLE design)
At the start: 37 parts, among them IC1 RP2040-QFN56, J1 N64_EDGE, Q1 BSS84, U4 MX66L1G45GMI-08GSOP_16L_300_M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

Commit message: 1Gbit pdf schematic
Parts:
- D1: value SL02-GS08DIODE_SL02-GS08_VIS-M -> SL02-GS08
- D3: value GREEN -> RED
- U4: value MX66L1G45GMI-08GSOP_16L_300_MAC-L -> MX66L1G45GMI-08G
Other:
- note added: "Do not solder R1 and D2 if LED3 is soldered."
- note removed: "Do not solder Q1 if D2 is soldered. Use either D2 or Q1. Do not solder R1 and R6."
- moved on the sheet: C11, C12, C13, C14, C22, C4, C7, D1, D2, D3, DEBUG, LED3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
