File: hw/n64cart-v3-soic-16.sch (EAGLE design)
At the start: 37 parts, among them IC1 RP2040-QFN56, J1 N64_EDGE, Q1 BSS84, U4 MX66L1G45GMI-08G

Commit message: missed pull down resistor for V3
Parts:
- added R6: 10K, rcl:R-EU_R0603
Connections:
- net +VBUS: now also R6.2
- net GND: now also R6.1
Changed lines of the file:
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@@
 <part name="D3" library="microbuilder" deviceset="LED" device="0603_NOOUTLINE" value="RED"/>
 <part name="D1" library="SL02-GS08" deviceset="SL02-GS08" device="DIODE_SL02-GS08_VIS-M" value="SL02-GS08"/>
+<part name="R6" library="rcl" library_urn="urn:adsk.eagle:library:334" deviceset="R-EU_" device="R0603" package3d_urn="urn:adsk.eagle:package:23555/3" value="10K"/>
+<part name="GND29" library="supply1" library_urn="urn:adsk.eagle:library:371" deviceset="GND" device=""/>
 </parts>
 <sheets>
@@
 <attribute name="VALUE" x="448.564" y="361.061" size="1.778" layer="96"/>
 </instance>
-<instance part="GND4" gate="1" x="447.04" y="345.44" smashed="yes">
-<attribute name="VALUE" x="444.5" y="342.9" size="1.778" layer="96"/>
+<instance part="GND4" gate="1" x="447.04" y="340.36" smashed="yes">
+<attribute name="VALUE" x="444.5" y="337.82" size="1.778" layer="96"/>
 </instance>
 <instance part="IC1" gate="IC$1" x="469.9" y="246.38" smashed="yes">
@@
 <attribute name="VALUE" x="336.7278" y="369.3668" size="1.778" layer="96" ratio="10" rot="SR0"/>
 <attribute name="NAME" x="341.3506" y="376.8344" size="1.778" layer="95" ratio="10" rot="SR0"/>
+</instance>
+<instance part="R6" gate="G$1" x="454.66" y="350.52" smashed="yes" rot="R90">
+<attribute name="NAME" x="453.1614" y="346.71" size="1.778" layer="95" rot="R90"/>
+<attribute name="VALUE" x="457.962" y="346.71" size="1.778" layer="96" rot="R90"/>
+</instance>
+<instance part="GND29" gate="1" x="454.66" y="340.36" smashed="yes">
+<attribute name="VALUE" x="452.12" y="337.82" size="1.778" layer="96"/>
 </instance>
 </instances>
@@
 <pinref part="C22" gate="G$1" pin="2"/>
 <pinref part="GND4" gate="1" pin="GND"/>
-<wire x1="447.04" y1="360.68" x2="447.04" y2="347.98" width="0.1524" layer="91"/>
+<wire x1="447.04" y1="360.68" x2="447.04" y2="342.9" width="0.1524" layer="91"/>
 </segment>
 <segment>
@@
 <pinref part="GND26" gate="1" pin="GND"/>
 <wire x1="236.22" y1="208.28" x2="236.22" y2="205.74" width="0.1524" layer="91"/>
+</segment>
+<segment>
+<pinref part="GND29" gate="1" pin="GND"/>
+<pinref part="R6" gate="G$1" pin="1"/>
+<wire x1="454.66" y1="342.9" x2="454.66" y2="345.44" width="0.1524" layer="91"/>
 </segment>
 </net>
@@
 <wire x1="454.66" y1="358.14" x2="454.66" y2="368.3" width="0.1524" layer="91"/>
 <label x="434.34" y="358.14" size="1.27" layer="95" rot="R180" xref="yes"/>
-</segment>
-<segment>
+<pinref part="R6" gate="G$1" pin="2"/>
+<wire x1="454.66" y1="355.6" x2="454.66" y2="358.14" width="0.1524" layer="91"/>
+<junction x="454.66" y="358.14"/>
+</segment>
+<segment>
